File: panel/TapOMatic_FrontPanel.kicad_pcb (KiCad board)
At the start: 2 copper layers, 121.6 x 128.4 mm, 0 parts

Commit message: full changes for second iteration
Other:
- board size 121.6 x 128.4 mm -> 121.6 x 128.5 mm

Commit message: adding text to back mask layer
Other:
- board text added: "Tap-O-Matic Divkid Discord Version, 2025"
